Commit message: Don't rotate legs frames relative to base

File: quad_vis/urdf/robot.urdf (robot description, URDF)
Before this commit: robot Quadrupel, 21 links, 20 joints
Joints:
- joint base_to_front_left_base: origin xyz=0.046 0.05 0 rpy=0 0 1.5708 -> xyz=0.046 0.05 0 rpy=0 0 0
- joint base_to_front_right_base: origin xyz=0.046 -0.05 0 rpy=0 0 -1.5708 -> xyz=0.046 -0.05 0 rpy=0 0 0
- joint base_to_rear_left_base: origin xyz=-0.046 0.05 0 rpy=0 0 1.5708 -> xyz=-0.046 0.05 0 rpy=0 0 0
- joint base_to_rear_right_base: origin xyz=-0.046 -0.05 0 rpy=0 0 -1.5708 -> xyz=-0.046 -0.05 0 rpy=0 0 0
- joint front_left_base_to_front_left_link1: limit lower=-1.7508 upper=1.7508 effort=1000.0 velocity=0.5 -> lower=0 upper=3.141592653589793 effort=1000.0 velocity=0.5
- joint front_right_base_to_front_right_link1: limit lower=-1.7508 upper=1.7508 effort=1000.0 velocity=0.5 -> lower=-3.141592653589793 upper=0 effort=1000.0 velocity=0.5
- joint rear_left_base_to_rear_left_link1: limit lower=-1.7508 upper=1.7508 effort=1000.0 velocity=0.5 -> lower=0 upper=3.141592653589793 effort=1000.0 velocity=0.5
- joint rear_right_base_to_rear_right_link1: limit lower=-1.7508 upper=1.7508 effort=1000.0 velocity=0.5 -> lower=-3.141592653589793 upper=0 effort=1000.0 velocity=0.5

Commit message: Put robot description in global package

File: quad_vis/urdf/robot.urdf (robot description, URDF)
Before this commit: robot Quadrupel, 21 links, 20 joints
Joints:
- joint base_to_front_left_base: origin xyz=0.046 0.05 0 rpy=0 0 0 -> xyz=0.046 0.06 0 rpy=0 0 0
- joint base_to_front_right_base: origin xyz=0.046 -0.05 0 rpy=0 0 0 -> xyz=0.046 -0.06 0 rpy=0 0 0
- joint base_to_rear_left_base: origin xyz=-0.046 0.05 0 rpy=0 0 0 -> xyz=-0.046 0.06 0 rpy=0 0 0
- joint base_to_rear_right_base: origin xyz=-0.046 -0.05 0 rpy=0 0 0 -> xyz=-0.046 -0.06 0 rpy=0 0 0

Commit message: Update legs parameters and fix leg urdf

File: quad_vis/urdf/robot.urdf (robot description, URDF)
Before this commit: robot Quadrupel, 21 links, 20 joints
Links:
- link front_left_link_2: geometry visual box size=0.07 0.02 0.02
- link front_right_link_2: geometry visual box size=0.07 0.02 0.02
- link rear_left_link_2: geometry visual box size=0.07 0.02 0.02
- link rear_right_link_2: geometry visual box size=0.07 0.02 0.02
Joints:
- joint front_left_link2_to_front_left_link3: origin xyz=0.067 0.0 0.0 rpy=0.0 -0.0 0.0 -> xyz=0.07 0.0 0.0 rpy=0.0 -0.0 0.0
- joint front_left_link3_to_front_left_link4: origin xyz=0.067 0.0 0.0 rpy=0.0 -0.0 0.0 -> xyz=0.05 0.0 0.0 rpy=0.0 -0.0 0.0
- joint front_right_link2_to_front_right_link3: origin xyz=0.067 0.0 0.0 rpy=0.0 -0.0 0.0 -> xyz=0.07 0.0 0.0 rpy=0.0 -0.0 0.0
- joint front_right_link3_to_front_right_link4: origin xyz=0.067 0.0 0.0 rpy=0.0 -0.0 0.0 -> xyz=0.05 0.0 0.0 rpy=0.0 -0.0 0.0
- joint rear_left_link2_to_rear_left_link3: origin xyz=0.067 0.0 0.0 rpy=0.0 -0.0 0.0 -> xyz=0.07 0.0 0.0 rpy=0.0 -0.0 0.0
- joint rear_left_link3_to_rear_left_link4: origin xyz=0.067 0.0 0.0 rpy=0.0 -0.0 0.0 -> xyz=0.05 0.0 0.0 rpy=0.0 -0.0 0.0
- joint rear_right_link2_to_rear_right_link3: origin xyz=0.067 0.0 0.0 rpy=0.0 -0.0 0.0 -> xyz=0.07 0.0 0.0 rpy=0.0 -0.0 0.0
- joint rear_right_link3_to_rear_right_link4: origin xyz=0.067 0.0 0.0 rpy=0.0 -0.0 0.0 -> xyz=0.05 0.0 0.0 rpy=0.0 -0.0 0.0
